File: PTP_Ante_Leko_Projekt1/PTP_Ante_Leko_Projekt1.kicad_pcb (KiCad board)
At the start: 2 copper layers, 45 parts, among them J1 Screw_Terminal_01x02, SW1 SW_MEC_5G, SW2 SW_SPDT_312, U1 LM2574N-5, U2 4027, U3 4027, U4 74LS47, U5 HDSP-7401, U7 NE555P

Commit message: lv7(ili 8)
Parts:
- moved SW1 42.8 mm to (147.2, 127.8)
- moved J1 16.4 mm to (214.9, 136.0)
- moved R13 13.8 mm to (176.2, 124.8)
- moved L1 10.3 mm to (196.5, 136.5)
- moved D5 7.79 mm to (221.2, 126.2), turned to 180 degrees
- moved D1 7.79 mm to (221.2, 102.0), turned to 180 degrees
- moved D2 7.79 mm to (221.2, 110.0), turned to 180 degrees
- moved D3 7.79 mm to (221.2, 118.0), turned to 180 degrees
- turned C5 to 180 degrees
- turned R19 to 0 degrees
Routing:
- net +5V: track 0.00 -> 188.2 mm, vias 0 -> 2
- net GND: track 0.00 -> 139.8 mm, vias 0 -> 1
- net Q1: track 0.00 -> 83.0 mm, vias 0 -> 4
- net Q0: track 0.00 -> 82.7 mm
- net Q2: track 0.00 -> 61.3 mm, vias 0 -> 3
- net Net-(D4-K): track 0.00 -> 45.7 mm
- net Net-(U3B-J): track 0.00 -> 42.8 mm
- net Net-(U7-THR): track 0.00 -> 33.4 mm, vias 0 -> 1
- net VD: track 1.00 -> 33.1 mm
- net Net-(U2B-J): track 0.00 -> 31.2 mm, vias 0 -> 2
- net Net-(U3A-J): track 0.00 -> 28.8 mm
- net Net-(U5-E): track 0.00 -> 27.6 mm
- net Net-(U4-BI): track 0.00 -> 26.9 mm, vias 0 -> 2
- net 555: track 0.00 -> 25.9 mm
- net Net-(U5-C): track 0.00 -> 24.8 mm, vias 0 -> 1
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- added copper zone on B.Cu, net GND

Commit message: lv8
Routing:
- net Clock: track 0.00 -> 77.6 mm, vias 0 -> 2
- net +5V: track 188.2 -> 258.3 mm
- net Reset: track 0.00 -> 61.0 mm, vias 0 -> 2
- net Q3: track 22.9 -> 54.1 mm, vias 0 -> 3
- net VD: track 33.1 -> 32.0 mm
- net Net-(U3B-J): track 42.8 -> 43.9 mm
Other:
- board outline added: 100 x 80 mm
- board text added: "Leko-BCD counter"
